File: OPL3_breakout.kicad_pcb (KiCad board)
At the start: 4 copper layers, 50 x 28.9 mm, 7 parts, among them J1 Conn_01x10, J2 Conn_01x10, J3 Conn_01x02, J4 Conn_01x02, U1 YMF262-M, U2 YAC512-M

Commit message: add test points
Parts:
- added TP1: DOAB, TestPoint:TestPoint_Keystone_5000-5004_Miniature, F.Cu at (163.5, 94.0)
- added TP2: CLK, TestPoint:TestPoint_Keystone_5000-5004_Miniature, F.Cu at (160.0, 94.0)
- added TP3: TST2, TestPoint:TestPoint_Keystone_5000-5004_Miniature, F.Cu at (177.5, 94.0)
- added TP4: TEST, TestPoint:TestPoint_Keystone_5000-5004_Miniature, F.Cu at (133.0, 107.0)
- added TP5: SMP2, TestPoint:TestPoint_Keystone_5000-5004_Miniature, F.Cu at (154.0, 105.5)
- added TP6: SMP1, TestPoint:TestPoint_Keystone_5000-5004_Miniature, F.Cu at (150.5, 105.5)
Connections:
- U1 pad 9: (no net) -> Net-(TP4-Pad1)
- U2 pad 15: (no net) -> Net-(TP3-Pad1)
Routing:
- net Net-(TP5-Pad1): track 23.6 -> 41.6 mm
- net Net-(TP2-Pad1): track 24.1 -> 35.6 mm
- net Net-(TP1-Pad1): track 31.1 -> 42.3 mm
- net Net-(TP6-Pad1): track 23.6 -> 33.7 mm
- net Net-(TP4-Pad1): track 0.00 -> 9.39 mm, vias 0 -> 1
- net Net-(TP3-Pad1): track 0.00 -> 4.01 mm
